Commit message: Fix Gazebo-real robot compatibility for SLAM Toolbox
- Update URDF frame names: remove robot2/ prefixes to match real robot
- Fix mesh file paths for current directory structure
- Create separate Gazebo navigation parameters with use_sim_time: true
- Update controller configuration for new frame naming
- Ensure frame consistency between simulation and real robot implementation

🤖 Generated with [Claude Code](https://claude.ai/code)

Co-Authored-By: Claude <noreply@anthropic.com>

File: yahboomcar_description/urdf/yahboomcar_robot2_gazebo.urdf (robot description, URDF)
Before this commit: robot yahboomcar, 8 links, 7 joints
Links:
- removed link robot2/base_footprint
- removed link robot2/base_link
- removed link robot2/imu_link
- removed link robot2/laser
- removed link robot2/left_back_wheel
- removed link robot2/left_front_wheel
- removed link robot2/right_back_wheel
- removed link robot2/right_front_wheel
- added link base_footprint
- added link base_link, mass 0.472828691870721; collision mesh filename=/home/mike/projects/b4m_yahboom/yahboomcar_description/mesh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; visual mesh filename=/home/mike/projects/b4m_yahboom/yahboomcar_description/mesh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
- added link imu_link, mass 0.0359997241016587; collision mesh filename=/home/mike/projects/b4m_yahboom/yahboomcar_description/mesh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; visual mesh filename=/home/mike/projects/b4m_yahboom/yahboomcar_description/mesh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
- added link laser, mass 0.0384696767042416; collision mesh filename=/home/mike/projects/b4m_yahboom/yahboomcar_description/mesh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; visual mesh filename=/home/mike/projects/b4m_yahboom/yahboomcar_description/mesh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
- added link left_back_wheel, mass 0.0500046612532973; collision mesh filename=/home/mike/projects/b4m_yahboom/yahboomcar_description/mesh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; visual mesh filename=/home/mike/projects/b4m_yahboom/yahboomcar_description/mesh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
- added link left_front_wheel, mass 0.0500162120573925; collision mesh filename=/home/mike/projects/b4m_yahboom/yahboomcar_description/mesh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; visual mesh filename=/home/mike/projects/b4m_yahboom/yahboomcar_description/mesh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
- added link right_back_wheel, mass 0.0500162120573925; collision mesh filename=/home/mike/projects/b4m_yahboom/yahboomcar_description/mesh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; visual mesh filename=/home/mike/projects/b4m_yahboom/yahboomcar_description/mesh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
- added link right_front_wheel, mass 0.0500047416034941; collision mesh filename=/home/mike/projects/b4m_yahboom/yahboomcar_description/mesh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; visual mesh filename=/home/mike/projects/b4m_yahboom/yahboomcar_description/mesh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
Joints:
- removed joint robot2/base_joint
- removed joint robot2/imu_joint
- removed joint robot2/left_back_joint
- removed joint robot2/left_front_joint
- removed joint robot2/lidar_joint
- removed joint robot2/right_back_joint
- removed joint robot2/right_front_joint
- added joint base_joint: type fixed, parent base_footprint, child base_link, origin xyz=0.0 0.0 0.0815 rpy=0 0 0
- added joint imu_joint: type fixed, parent base_link, child imu_link, origin xyz=-0.00080703 0.0418 0.040805 rpy=0 0 0, axis 0 0 0
- added joint left_back_joint: type continuous, parent base_link, child left_back_wheel, origin xyz=-0.06 0.083967 -0.03295 rpy=0 0 0, axis 0 1 0
- added joint left_front_joint: type continuous, parent base_link, child left_front_wheel, origin xyz=0.06 0.08361 -0.03295 rpy=0 0 0, axis 0 1 0
- added joint lidar_joint: type fixed, parent base_link, child laser, origin xyz=-0.0019517 0.00040736 0.12059 rpy=0 0 0, axis 0 0 0
- added joint right_back_joint: type continuous, parent base_link, child right_back_wheel, origin xyz=-0.06 -0.08361 -0.03295 rpy=0 0 0, axis 0 1 0
- added joint right_front_joint: type continuous, parent base_link, child right_front_wheel, origin xyz=0.06 -0.08361 -0.03295 rpy=0 0 0, axis 0 1 0

Commit message: Fix robot model for Ignition Gazebo ground contact and wheel physics
- Adjust base_joint height from 0.0815m to 0.06595m for proper wheel-ground contact
- Replace mesh-based wheel collisions with cylinder geometry (radius=0.033m, length=0.015m)
- Properly orient wheel cylinders with rpy="1.57079632679 0 0"
- Ensures all 4 wheels have accurate physics collision for simulation

🤖 Generated with [Claude Code](https://claude.ai/code)

Co-Authored-By: Claude <noreply@anthropic.com>

File: yahboomcar_description/urdf/yahboomcar_robot2_gazebo.urdf (robot description, URDF)
Before this commit: robot yahboomcar, 8 links, 7 joints
Links:
- link left_back_wheel: geometry collision cylinder length=0.015 radius=0.033; visual mesh filename=/home/mike/projects/b4m_yahboom/yahboomcar_description/mesh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
- link left_front_wheel: geometry collision cylinder length=0.015 radius=0.033; visual mesh filename=/home/mike/projects/b4m_yahboom/yahboomcar_description/mesh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
- link right_back_wheel: geometry collision cylinder length=0.015 radius=0.033; visual mesh filename=/home/mike/projects/b4m_yahboom/yahboomcar_description/mesh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
- link right_front_wheel: geometry collision cylinder length=0.015 radius=0.033; visual mesh filename=/home/mike/projects/b4m_yahboom/yahboomcar_description/mesh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
Joints:
- joint base_joint: origin xyz=0.0 0.0 0.0815 rpy=0 0 0 -> xyz=0.0 0.0 0.06595 rpy=0 0 0

Commit message: Fix robot turning in Ignition Gazebo simulation
- Fixed wheel-ground friction parameters (mu1=100.0, mu2=100.0 for drive wheels)
- Corrected wheel separation to 0.167m in differential drive plugin
- Increased robot mass to 1.5kg and improved inertial properties
- Set back wheels as low-friction casters (mu1=0.1, mu2=0.1)
- Fixed ROS-Ignition bridge syntax (@ instead of ] and [)
- Removed conflicting ros2_control spawners for direct DiffDrive
- Added comprehensive tests for square navigation with corner tracking
- Robot now successfully completes 1-meter square navigation test

🤖 Generated with [Claude Code](https://claude.ai/code)

Co-Authored-By: Claude <noreply@anthropic.com>

File: yahboomcar_description/urdf/yahboomcar_robot2_gazebo.urdf (robot description, URDF)
Before this commit: robot yahboomcar, 8 links, 7 joints
Links:
- link base_link: mass 0.472828691870721 -> 1.5
Joints:
- joint left_back_joint: limit (none) -> effort=100 velocity=100
- joint left_front_joint: limit (none) -> effort=100 velocity=100
- joint right_back_joint: limit (none) -> effort=100 velocity=100
- joint right_front_joint: limit (none) -> effort=100 velocity=100
